Commit message: [fix] audit: add imu_link to URDF, imu.launch.py, LICENSE, .gitignore, imp2_safety + imp2_diagnostics console_scripts + 3 node stubs (estop_bridge, heartbeat_monitor, safety_state, battery_monitor, cpu_temp_monitor), SYSTEM_DEPS.md

File: src/imp2_description/urdf/imp2.xacro (robot description, xacro)
@@ -109,4 +109,19 @@
     <origin xyz="0 0 0" rpy="0 0 0" />
   </joint>
+  <!-- BNO085 IMU (ADR-0012)
+       Mounted on top layer (warstwa 3), central, 80mm from motors.
+       Per ADR-0008: 10 cm above base_link, X-fwd convention. -->
+  <link name="imu_link">
+    <inertial>
+      <mass value="0.005" />  <!-- BNO085 is ~5g -->
+      <origin xyz="0 0 0" />
+      <inertia ixx="0.0001" ixy="0" ixz="0" iyy="0.0001" iyz="0" izz="0.0001" />
+    </inertial>
+  </link>
+  <joint name="base_to_imu" type="fixed">
+    <parent link="base_link" />
+    <child link="imu_link" />
+    <origin xyz="0 0 0.10" rpy="0 0 0" />
+  </joint>
   <!-- ros2_control: micro-ROS hardware interface -->
   <ros2_control name="imp2_hw" type="system">
